Commit message: Renamed file and fixed gripper

File: lynxmotion/al5d.urdf (robot description, URDF)
Before this commit: robot al5d_arm, 7 links, 6 joints
Links:
- added link tool_center_point; visual box size=0.005 0.005 0.005
Joints:
- added joint center_point: type fixed, parent hand, child tool_center_point, origin xyz=0.075 0 0 rpy=0 0 0
- joint left_gripper: type prismatic -> fixed
- joint right_gripper: type prismatic -> fixed
